File: KiCAD/AddressDecoder.kicad_sch (KiCad schematic)
At the start: 11 parts

Commit message: Update schematics
- Bugfixes for addressing
- Adding more info on PAL in video circuit
Other:
- note added: "3000..33FF"
- note added: "3400..37FF"
- note removed: "3000..34FF"
- note removed: "3400..38FF"
Changed lines of the file:
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@@
 	(title_block
 		(title "TRS-80 Model I Rev HE11E011550")
-		(date "2025-06-14")
+		(date "2025-06-15")
 		(rev "E1A")
 		(company "RetroStack - Marcel Erz")
@@
 		)
 	)
-	(text "3000..34FF"
+	(text "3000..33FF"
 		(exclude_from_sim no)
 		(at 98.425 117.475 0)
@@
 		)
 	)
-	(text "3400..38FF"
+	(text "3400..37FF"
 		(exclude_from_sim no)
 		(at 98.425 120.015 0)
@@
 	)
 	(junction
+		(at 193.04 102.235)
+		(diameter 0)
+		(color 0 0 0 0)
+	)
+	(junction
+		(at 135.255 102.235)
+		(diameter 0)
+		(color 0 0 0 0)
+	)
+	(junction
 		(at 146.685 117.475)
 		(diameter 0)
@@
 	)
 	(junction
-		(at 141.224 102.235)
-		(diameter 0)
-		(color 0 0 0 0)
-	)
-	(junction
 		(at 59.055 67.945)
 		(diameter 0)
@@
 	)
 	(junction
+		(at 196.215 97.155)
+		(diameter 0)
+		(color 0 0 0 0)
+	)
+	(junction
 		(at 163.449 97.155)
 		(diameter 0)
@@
 	)
 	(junction
-		(at 193.421 102.362)
+		(at 141.605 102.235)
 		(diameter 0)
 		(color 0 0 0 0)
@@
 	(junction
 		(at 136.525 84.455)
-		(diameter 0)
-		(color 0 0 0 0)
-	)
-	(junction
-		(at 196.469 97.155)
 		(diameter 0)
 		(color 0 0 0 0)
@@
 		)
 	)
+	(wire
+		(pts
+			(xy 193.04 117.475) (xy 201.93 117.475)
+		)
+		(stroke
+			(width 0)
+			(type default)
+		)
+	)
 	(bus
 		(pts
@@
 		)
 	)
-	(wire
-		(pts
-			(xy 193.421 117.475) (xy 193.421 102.362)
-		)
-		(stroke
-			(width 0)
-			(type default)
-		)
-	)
 	(bus
 		(pts
@@
 	(wire
 		(pts
-			(xy 180.34 97.155) (xy 196.469 97.155)
+			(xy 180.34 97.155) (xy 196.215 97.155)
 		)
 		(stroke
@@
 	(wire
 		(pts
-			(xy 196.469 97.155) (xy 196.469 114.935)
+			(xy 196.215 97.155) (xy 196.215 114.935)
 		)
 		(stroke
@@
 	(wire
 		(pts
-			(xy 201.93 114.935) (xy 196.469 114.935)
+			(xy 201.93 114.935) (xy 196.215 114.935)
 		)
 		(stroke
@@
 		)
 	)
+	(wire
+		(pts
+			(xy 141.605 102.235) (xy 193.04 102.235)
+		)
+		(stroke
+			(width 0)
+			(type default)
+		)
+	)
 	(bus
 		(pts
@@
 	(wire
 		(pts
-			(xy 141.605 102.235) (xy 141.224 102.235)
+			(xy 135.255 102.235) (xy 141.605 102.235)
 		)
 		(stroke
@@
 	(wire
 		(pts
-			(xy 141.224 102.362) (xy 193.421 102.362)
-		)
-		(stroke
-			(width 0)
-			(type default)
-		)
-	)
-	(wire
-		(pts
 			(xy 158.496 65.405) (xy 238.125 65.405)
 		)
@@
 	(wire
 		(pts
+			(xy 135.001 102.235) (xy 135.255 102.235)
+		)
+		(stroke
+			(width 0)
+			(type default)
+		)
+	)
+	(wire
+		(pts
 			(xy 141.605 84.455) (xy 141.605 85.09)
 		)
@@
 	(wire
 		(pts
-			(xy 141.224 102.362) (xy 141.224 102.235)
-		)
-		(stroke
-			(width 0)
-			(type default)
-		)
-	)
-	(wire
-		(pts
 			(xy 146.685 84.455) (xy 141.605 84.455)
 		)
@@
 	(wire
 		(pts
-			(xy 135.255 102.235) (xy 141.224 102.235)
-		)
-		(stroke
-			(width 0)
-			(type default)
-		)
-	)
-	(wire
-		(pts
 			(xy 55.88 67.945) (xy 59.055 67.945)
 		)
@@
 	(wire
 		(pts
-			(xy 201.93 117.475) (xy 193.421 117.475)
-		)
-		(stroke
-			(width 0)
-			(type default)
-		)
-	)
-	(wire
-		(pts
 			(xy 135.255 117.475) (xy 146.685 117.475)
 		)
@@
 	(wire
 		(pts
-			(xy 238.125 97.155) (xy 196.469 97.155)
-		)
-		(stroke
-			(width 0)
-			(type default)
-		)
-	)
-	(wire
-		(pts
 			(xy 107.315 104.775) (xy 107.315 111.125)
 		)
@@
 	(wire
 		(pts
-			(xy 193.421 102.235) (xy 238.125 102.235)
-		)
-		(stroke
-			(width 0)
-			(type default)
-		)
-	)
-	(wire
-		(pts
 			(xy 97.79 99.695) (xy 118.745 99.695)
 		)
@@
 	(wire
 		(pts
+			(xy 193.04 102.235) (xy 238.125 102.235)
+		)
+		(stroke
+			(width 0)
+			(type default)
+		)
+	)
+	(wire
+		(pts
 			(xy 84.455 62.865) (xy 86.995 62.865)
 		)
@@
 	(wire
 		(pts
-			(xy 193.421 102.235) (xy 193.421 102.362)
+			(xy 196.215 97.155) (xy 238.125 97.155)
+		)
+		(stroke
+			(width 0)
+			(type default)
+		)
+	)
+	(wire
+		(pts
+			(xy 193.04 102.235) (xy 193.04 117.475)
 		)
 		(stroke
@@
 				)
 			)
-			(table_cell "-"
+			(table_cell "X"
 				(exclude_from_sim no)
 				(at 127 132.08 0)
@@
 				)
 			)
-			(table_cell "-"
+			(table_cell "X"
 				(exclude_from_sim no)
 				(at 132.08 132.08 0)
@@
 				)
 			)
-			(table_cell "-"
+			(table_cell "X"
 				(exclude_from_sim no)
 				(at 137.16 132.08 0)
@@
 				)
 			)
-			(table_cell "X"
+			(table_cell "-"
 				(exclude_from_sim no)
 				(at 127 134.62 0)
@@
 				)
 			)
-			(table_cell "X"
+			(table_cell "-"
 				(exclude_from_sim no)
 				(at 132.08 134.62 0)
@@
 				)
 			)
-			(table_cell "-"
+			(table_cell "X"
 				(exclude_from_sim no)
 				(at 137.16 134.62 0)
@@
 				)
 			)
-			(table_cell "X"
+			(table_cell "-"
 				(exclude_from_sim no)
 				(at 127 137.16 0)
@@
 				)
 			)
-			(table_cell "X"
+			(table_cell "-"
 				(exclude_from_sim no)
 				(at 132.08 137.16 0)
@@
 				)
 			)
-			(table_cell "X"
+			(table_cell "-"
 				(exclude_from_sim no)
 				(at 137.16 137.16 0)
